File: PCB/board - Copy/E155 Development Board/E155 Development Board.kicad_sch (KiCad schematic)
At the start: 48 parts, among them J1 Screw_Terminal_01x02, J2 ESP RST Jumper, J3 FPGA Jumper, J4 MCU Jumper, J5 3V7 Lipo 1, J6 3V7 Lipo 2, Q1 2N3906, SW4 SW_Push, SW5 SW_Push, SW6 SW_Push, SW7 SW_DIP_x08, U1 NUCLEO-LxxxKx, U2 UPduino_v3.1, U3 LD1117DT50TR, U4 LD1117DT33CTR, U5 mikroBUS_SOCKET, U6 LM386, U7 TSSP6P38, U8 TSSP6P38, U9 TSSP6P38

Commit message: Added Flash LED
Parts:
- removed J5: 3V7 Lipo 1, Connector_JST:JST_PH_B2B-PH-K_1x02_P2.00mm_Vertical, symbol Connector_Generic:Conn_01x02
- removed U8, U9: TSSP6P38, OptoDevice:Vishay_MINICAST-3Pin, symbol Sensor_Proximity:TSSP58038
- added D5: R(or B) LED, LED_SMD:LED_0805_2012Metric_Pad1.15x1.40mm_HandSolder, symbol Device:LED
- added R12, R13: 330, Resistor_SMD:R_0805_2012Metric_Pad1.20x1.40mm_HandSolder, symbol Device:R_US
- J6: value 3V7 Lipo 2 -> 2S Lipo
- SW6: value SW_Push -> Trigger
- U7: value TSSP6P38 -> TSOP38238
Connections:
- net BATT_MID is gone; now on net BATT: J6.1 (Pin_1)
- net FPGA Pin is gone; now on net P37: R11.2, SW6.2
- net +3V3: now also R11.1
- net +5V: no longer R11.1
- net GND: now also R12.2
- net P10: now also SW7.11
- net P12: now also SW7.10
- net P20: now also SW7.12
- net P21: now also SW7.9
- net P23: now also SW7.15
- net P27: now also SW7.16
- net P32: now also U7.1 (OUT)
- net P34: now also R13.2
- net P43: now also D5.2 (A)
- net PA11: now also SW7.5
- net PA6: now also SW7.1
- net PB3: now also SW7.8
- net PB4: now also SW7.7
- net PB5: now also SW7.6
- net TBD: no longer SW7.1, SW7.10, SW7.11, SW7.12, SW7.15, SW7.16, SW7.5, SW7.6, SW7.7, SW7.8, SW7.9
- net FPGA PIN: no longer names the net of Q1.2 (B)
- net FPGA PIN: now also R13.1; no longer U7.1 (OUT)
- new net: D5.1 (K), R12.1
Other:
- note added: "MCU CS"
- note added: "MCU MISO"
- note added: "MCU MOSI"
- note added: "MCU SCK"
- moved on the sheet: R11, SW6, U7

Commit message: Labels for IR schematic
Other:
- note added: "Flash"
- note added: "IR Led"
- note added: "IR Reciever"
- note added: "Trigger"
Changed lines of the file:
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@@
+		)
+	)
+	(text "Flash"
+		(exclude_from_sim no)
+		(at 170.688 213.868 0)
+		(effects
+			(font
+				(size 1.27 1.27)
+			)
 		)
 	)
@@
 		)
 	)
+	(text "IR Reciever"
+		(exclude_from_sim no)
+		(at 221.742 219.456 0)
+		(effects
+			(font
+				(size 1.27 1.27)
+			)
+		)
+	)
 	(text "Mounting Holes"
 		(exclude_from_sim no)
@@
 		)
 	)
+	(text "Trigger"
+		(exclude_from_sim no)
+		(at 192.532 213.36 0)
+		(effects
+			(font
+				(size 1.27 1.27)
+			)
+		)
+	)
 	(text "Bridge Connector"
 		(exclude_from_sim no)
@@
 			)
 		)
+	)
+	(text "IR Led"
+		(exclude_from_sim no)
+		(at 116.332 207.772 0)
+		(effects
+			(font
+				(size 1.27 1.27)
+			)
+		)

Commit message: Added Schematic V1 and Board changes
Parts:
- removed J1: Screw_Terminal_01x02, TerminalBlock_Phoenix:TerminalBlock_Phoenix_MKDS-1,5-2-5.08_1x02_P5.08mm_Horizontal, symbol Connector:Screw_Terminal_01x02
- removed SW7: SW_DIP_x08, Button_Switch_THT:SW_DIP_SPSTx08_Slide_6.7x21.88mm_W7.62mm_P2.54mm_LowProfile, symbol Switch:SW_DIP_x08
- added D6: LED, LED_SMD:LED_0805_2012Metric_Pad1.15x1.40mm_HandSolder, symbol Device:LED
- added R14: 1.2k, Resistor_SMD:R_0805_2012Metric_Pad1.20x1.40mm_HandSolder, symbol Device:R_US
- added R15: 330, Resistor_SMD:R_0805_2012Metric_Pad1.20x1.40mm_HandSolder, symbol Device:R_US
- added SW1: KCD11 Rocker, symbol Switch:SW_SPST
- added TP1: BATT_RAW, TestPoint:TestPoint_Pad_2.0x2.0mm, symbol Connector:TestPoint
- C6: value C_Small -> 0.1uF
- C8: value 250uF -> 220uF
- R10: value 1k -> 100
Connections:
- net MCU PIN is gone; now on net PA4: R9.1
- net PA11 is gone; now on net P20: U1.13 (D10/PA11/CS), U5.3 (CS)
- net PB3 is gone; now on net P21: U1.16 (D13/PB3/SCK), U5.4 (SCK)
- net PB4 is gone; now on net P12: U1.15 (D12/PB4/MISO), U5.5 (MISO)
- net PB5 is gone; now on net P10: U1.14 (D11/PB5/MOSI), U5.6 (MOSI)
- net BATT: now also SW1.2 (B); no longer J6.1 (Pin_1)
- net GND: now also R15.2
- net P13: now also D6.2 (A)
- net at C5.1: now also R14.1; no longer U6.1 (GAIN)
- new net: R14.2, U6.1 (GAIN)
- new net: D6.1 (K), R15.1
- new net BATT_RAW: J6.1 (Pin_1), SW1.1 (A), TP1.1
- no-connect marks 14 -> 44
Other:
- note added: "3A Rocker Switch"
- note added: "IR Flash"
- note added: "IR Receiver"
- note added: "SPI Connections"
- note added: "Test Points"
- note removed: "Battery Management"
- note removed: "Bridge Connector"
- note removed: "Do we need more LED indicators?"
- note removed: "Fix this transistor setup"
- note removed: "IR Led"
- note removed: "IR Reciever"
- note removed: "Power Input Screw Terminal"
- title: E155 Development Board -> MicroPs Project
- moved on the sheet: C1, C2, C3, C4, C5, C6, C7, C8, D1, D2, D3, D4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

Commit message: Cleaning up PCB
Parts:
- J2: footprint (none) -> Connector_PinHeader_2.54mm:PinHeader_1x02_P2.54mm_Vertical
Changed lines of the file:
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@@
 			)
 		)
-		(property "Footprint" ""
+		(property "Footprint" "Connector_PinHeader_2.54mm:PinHeader_1x02_P2.54mm_Vertical"
 			(at 226.06 46.99 0)
 			(hide yes)
