File: PCB/board - Copy/E155 Development Board/E155 Development Board.kicad_pcb (KiCad board)
At the start: 2 copper layers, 106.9 x 105.3 mm, 48 parts, among them J1 Screw_Terminal_01x02, J2 Conn_01x03, J3 Conn_01x02, J4 Conn_01x02, J6 Conn_02x20_Odd_Even, J7 Conn_01x06, SW0 SW_Push, SW1 SW_Push, SW2 SW_Push, SW3 SW_Push, SW4 SW_Push, SW5 SW_Push, SW6 SW_DIP_x04, SW7 SW_DIP_x08, U1 NUCLEO-LxxxKx, U2 UPduino_v3.1, U3 LD1117DT50TR, U4 LD1117DT33CTR, U5 mikroBUS_SOCKET

Commit message: Cleaning up PCB
Parts:
- removed D7, D8: LED (B), LED_SMD:LED_0805_2012Metric_Pad1.15x1.40mm_HandSolder
- removed J1: Screw_Terminal_01x02, TerminalBlock_Phoenix:TerminalBlock_Phoenix_MKDS-1,5-2-5.08_1x02_P5.08mm_Horizontal
- removed J7: Conn_01x06, Connector_PinSocket_2.54mm:PinSocket_1x06_P2.54mm_Vertical
- removed SW0, SW1, SW2, SW3: SW_Push, Button_Switch_THT:SW_PUSH_6mm_H4.3mm
- removed SW7: SW_DIP_x08, Button_Switch_THT:SW_DIP_SPSTx08_Slide_6.7x21.88mm_W7.62mm_P2.54mm_LowProfile
- added Q1: 2N3906, Package_TO_SOT_THT:TO-92_Inline, F.Cu at (194.5, 91.4)
- added R12: 330, Resistor_SMD:R_0805_2012Metric_Pad1.20x1.40mm_HandSolder, F.Cu at (202.8, 83.0)
- added R13: 330, Resistor_SMD:R_0805_2012Metric_Pad1.20x1.40mm_HandSolder, F.Cu at (202.8, 86.0)
- added R14: 1.2k, Resistor_SMD:R_0805_2012Metric_Pad1.20x1.40mm_HandSolder, F.Cu at (202.8, 88.9)
- added R15: 330, Resistor_SMD:R_0805_2012Metric_Pad1.20x1.40mm_HandSolder, F.Cu at (202.8, 91.9)
- added TP1: BATT_RAW, TestPoint:TestPoint_Pad_2.0x2.0mm, F.Cu at (207.2, 83.6)
- added U7: TSOP38238, OptoDevice:Vishay_MINICAST-3Pin, F.Cu at (204.7, 75.2)
- D3: value LED (G) -> LED (B)
- D4: value LED (G) -> IR LED
- D5: value LED (G) -> R(or B) LED
- D6: value LED (B) -> LED
- J2: value Conn_01x03 -> ESP RST Jumper; footprint Connector_PinHeader_2.54mm:PinHeader_1x03_P2.54mm_Vertical -> Connector_PinHeader_2.54mm:PinHeader_1x02_P2.54mm_Vertical
- J3: value Conn_01x02 -> FPGA Jumper
- J4: value Conn_01x02 -> MCU Jumper
- J6: value Conn_02x20_Odd_Even -> 2S Lipo; footprint E155_Footprints:2x20 Pin Header Keyed -> Connector_JST:JST_PH_B2B-PH-K_1x02_P2.00mm_Vertical
- R10: value 1k -> 100
- R11, R8, R9: value 1k -> 10k
- R7: value 1k -> 10
- SW6: value SW_DIP_x04 -> Trigger; footprint Button_Switch_THT:SW_DIP_SPSTx04_Slide_6.7x11.72mm_W7.62mm_P2.54mm_LowProfile -> Button_Switch_THT:SW_PUSH_6mm_H4.3mm
- moved J6 161.3 mm to (195.5, 84.3), turned to 0 degrees
- moved SW6 158.9 mm to (194.5, 75.0)
Connections:
- C1 pad 1: /VIN -> /BATT
- C3 pad 1: /VIN -> /BATT
- D1 pad 2: /VIN -> /BATT
- D2 pad 2: /PA10 -> +5V
- D3 pad 2: /PA9 -> +3V3
- D4 pad 2: /PA6 -> Net-(D4-A)
- D5 pad 2: /PB3 -> /P43
- D6 pad 2: /P42 -> /P13
- J6 pad 1: /VIN -> /BATT_RAW
- R10 pad 1: Net-(D7-K) -> Net-(D4-K)
- R11 pad 1: Net-(D8-K) -> +3V3
- R11 pad 2: GND -> /P37
- R7 pad 1: Net-(D4-K) -> Net-(C8-Pad2)
- R7 pad 2: GND -> Net-(C7-Pad1)
- R8 pad 1: Net-(D5-K) -> Net-(U6-+)
- R9 pad 1: Net-(D6-K) -> /PA4
- R9 pad 2: GND -> Net-(U6-+)
- SW6 pad 2: GND -> /P37
- U1 pad 13: /PA11 -> /P20
- U1 pad 14: /PB5 -> /P10
- U1 pad 15: /PB4 -> /P12
- U1 pad 16: /PB3 -> /P21
- U1 pad 26: /PA2 -> unconnected-(U1-A7/PA2-Pad26)
- U3 pad 3: /VIN -> /BATT
- U4 pad 3: /VIN -> /BATT
- U5 pad 3: /PA11 -> /P20
- U5 pad 4: /PB3 -> /P21
- U5 pad 5: /PB4 -> /P12
- U5 pad 6: /PB5 -> /P10
Routing:
- net /PA10: track 263.7 -> 62.1 mm, vias 8 -> 2
- net /PA6: track 189.4 -> 0.00 mm, vias 3 -> 0
- net /PA9: track 260.9 -> 73.0 mm, vias 2 -> 0
- net /P20: track 176.7 -> 0.00 mm, vias 2 -> 0
- net /P10: track 168.7 -> 0.00 mm, vias 2 -> 0
- net /P21: track 164.4 -> 0.00 mm, vias 2 -> 0
- net /PA12: track 159.6 -> 0.00 mm, vias 2 -> 0
- net /VIN: track 155.2 -> 0.00 mm, vias 3 -> 0
- net /P12: track 153.4 -> 0.00 mm, vias 2 -> 0
- net /PB3: track 146.5 -> 0.00 mm, vias 3 -> 0
- net /PA5: track 138.2 -> 0.00 mm, vias 1 -> 0
- net /PA11: track 134.1 -> 0.00 mm, vias 2 -> 0
- net /PB5: track 128.2 -> 0.00 mm, vias 2 -> 0
- net /PB4: track 122.1 -> 0.00 mm, vias 2 -> 0
- net +5V: track 120.0 -> 5.32 mm, vias 3 -> 0
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Other:
- board text removed: "P10"
- board text removed: "P11"
- board text removed: "P12"
- board text removed: "P13"
- board text removed: "P18"
- board text removed: "P19"
- board text removed: "P2"
- board text removed: "P20"
- board text removed: "P21"
- board text removed: "P23"
- board text removed: "P25"
- board text removed: "P26"
- board text removed: "P27"
- board text removed: "P3"
- board text removed: "P34"
- board text removed: "P36"
- board text removed: "P4"
- board text removed: "P43"
- board text removed: "P44"
- board text removed: "P45"
- board text removed: "P46"
- board text removed: "P47"
- board text removed: "P48"
- board text removed: "P6"
- board text removed: "P9"
- board text removed: "PA10 (RX)"
- board text removed: "PA11 (CS)"
- board text removed: "PA5 (SDA)"
- board text removed: "PA6 (SCL)"
- board text removed: "PA9 (TX)"
- board text removed: "PB1"
- board text removed: "PB3 (SCK)"
- board text removed: "PB4 (CIPO)"
- board text removed: "PB5 (COPI)"
- board text removed: "PMOD"

Commit message: random
Parts:
- removed D1: LED (R), LED_SMD:LED_0805_2012Metric_Pad1.15x1.40mm_HandSolder
- removed R4: 1k, Resistor_SMD:R_0805_2012Metric_Pad1.20x1.40mm_HandSolder
Routing:
- net Net-(D1-K): track 5.48 -> 0.00 mm

Commit message: board cleanup
Routing:
- net /~{FPGA_RESET}: track 108.1 -> 0.00 mm, vias 1 -> 0
- net +3V3: track 104.5 -> 0.99 mm, vias 4 -> 1
- net /BATT: track 73.7 -> 0.00 mm, vias 2 -> 0
- net /PA9: track 73.0 -> 0.00 mm
- net /MIKROBUS_RST: track 71.4 -> 0.00 mm
- net /FPGA_+5V: track 69.0 -> 0.00 mm
- net /MCU_+5V: track 62.6 -> 0.00 mm, vias 2 -> 0
- net /PA10: track 62.1 -> 0.00 mm, vias 2 -> 0
- net GND: track 32.6 -> 0.00 mm, vias 1 -> 0
- net /P28: track 30.3 -> 0.00 mm
- net /P38: track 30.0 -> 0.00 mm
- net /P42: track 29.6 -> 0.00 mm
- net /~{MCU_RESET}: track 20.0 -> 0.00 mm, vias 3 -> 0
- net Net-(D4-K): track 11.0 -> 0.00 mm
- net Net-(D6-K): track 5.48 -> 0.00 mm
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
Commit message: Board Rearrange
Parts:
- moved R1 62.4 mm to (39.5, 78.5), turned to 180 degrees
- moved SW4 62.1 mm to (42.8, 73.2)
- moved SW5 52.7 mm to (42.8, 88.2)
- moved R2 49.5 mm to (39.5, 94.0), turned to 180 degrees
- moved J2 21.9 mm to (83.8, 113.3)
- moved J4 21.9 mm to (90.0, 104.2)
- moved J3 21.9 mm to (83.8, 104.3)
- moved R3 21.9 mm to (87.3, 114.3)
- moved U5 16.4 mm to (103.1, 58.9)
- moved C1 15.0 mm to (126.7, 98.8)
- moved C2 15.0 mm to (104.9, 96.6)
- moved C3 15.0 mm to (110.3, 99.5)
- moved C4 15.0 mm to (130.7, 90.5)
- moved U3 15.0 mm to (125.5, 90.3)
- moved U4 15.0 mm to (110.3, 90.3)
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Routing:
- net Net-(J2-Pin_1): track 11.0 -> 0.00 mm
- net +3V3: track 0.99 -> 0.00 mm, vias 1 -> 0
Other:
- board text removed: "P28"
- board text removed: "P38"
- board text removed: "P42"
